Commit message: ms_robot+hospital

File: description/robot_core.xacro (robot description, xacro)
@@ -40,5 +40,5 @@
                 <box size="0.3 0.3 0.15"/>
             </geometry>
-            <material name="green"/>
+            <material name="orange"/>
         </visual>
         <collision>
@@ -53,5 +53,5 @@
     </link>
     <gazebo reference="chassis">
-        <material>Gazebo/Green</material>
+        <material>Gazebo/Orange</material>
     </gazebo>
     <!-- LEFT WHEEL LINK -->
